File: melzi.sch (EAGLE design)
At the start: 147 parts, among them IC1 A4988, IC2 A4988, IC3 A4988, IC4 A4988, IC5 7805DT, IC6 ATMEGA644A, IC7 4050D, IC8 FT232RL-BASICSSOP, M1 RFP30N06LE, M2 RFP30N06LE, M3 RFP30N06LE, Q1 16MHZ, T1 TRIM, T2 TRIM, T3 TRIM, T4 TRIM, U2 A4982, X1 MICROSD, X2 MINI-USB-SHIELD-UX60-MB-5ST

Commit message: Melzi update wip
Parts:
- removed C1: 100 uF, rcl:CPOL-EUUD-6,3X7,7
- removed C10, C11, C12, C33: .1uf, SparkFun:CAP0805
- removed C13, C34: .22uf, SparkFun:CAP0805
- removed IC1: A4988, allegro:A4983
- removed JP18: MOT-X, SparkFun:M04POLAR
- removed JS4: MS1, SparkFun:JUMPER-2SMD-NC
- removed JS5: MS2, SparkFun:JUMPER-2SMD-NC
- removed JS6: MS3, SparkFun:JUMPER-2SMD-NC
- removed R13: 100k, SparkFun:RESISTOR
- removed R14, R15: 10k, SparkFun:RESISTOR
- removed R6: 20k, SparkFun:RESISTOR
- removed S1, S2: 0.05, SparkFun:RESISTOR1206
- removed T1: TRIM, SparkFun:TRIMPOTSMD
- added JS16: MS3, SparkFun:JUMPER-2SMD-NC
- added R33: 200R, rcl:R-EU_0309/V
Connections:
- removed net !XY-ENABLE: R31.2, U2.!ENABLE
- removed net +5V: C48.2, MS-X.2, R31.1, R32.1, R39.2, U2.VDD
- removed net 12V: C49.1, C50.+, C51.1, U2.VBB1, U2.VBB2
- removed net N$18: IC1.MS3, JS6.1
- removed net N$19: IC1.MS2, JS5.1
- removed net N$3: IC1.MS1, JS4.1
- removed net XCP1: C10.1, IC1.CP1
- removed net XCP2: C10.2, IC1.CP2
- removed net XOUT1A: IC1.OUT1A, JP1.3
- removed net XOUT1B: IC1.OUT1B, JP1.4
- removed net XOUT2A: IC1.OUT2A, JP1.2
- removed net XOUT2B: IC1.OUT2B, JP1.1
- removed net XREF: IC1.REF, T1.WIPER
- removed net XREF2: R6.2, T1.CW
- removed net XROSC: IC1.ROSC, R14.1
- removed net XSENSE1: IC1.SENSE1, S2.2
- removed net XSENSE2: IC1.SENSE2, S1.2
- removed net XSLEEP: IC1.RESET, IC1.SLEEP, R15.2
- removed net XVCP: C33.2, IC1.VCP
- removed net XVREG: C34.2, IC1.VREG
- new net N$36: C26.1, IC5.VI, JS16.1, R33.1
- net !XYEENABLE: now also R31.2, U2.!ENABLE; no longer IC1.ENABLE, R13.2
- net GND: no longer C1.-, C11.2, C12.1, C13.2, C34.1, IC1.EXP, IC1.GND, IC1.GND@1, IC1.NC, IC1.NC@1, IC1.NC@2, R14.2, S1.1, S2.1, T1.CCW
- net N$32: now also JP1.3; no longer JP18.3
- net N$33: now also JP1.4; no longer JP18.4
- net N$34: now also JP1.2; no longer JP18.2
- net N$35: now also JP1.1; no longer JP18.1
- net VCC: now also C48.2, MS-X.2, R31.1, R32.1, R39.2, U2.VDD; no longer C13.1, IC1.VDD, JS4.2, JS5.2, JS6.2, R13.1, R15.1, R6.1
- net VMOT: now also C49.1, C50.+, C51.1, JS16.2, R33.2, U2.VBB1, U2.VBB2; no longer C1.+, C11.1, C12.2, C26.1, C33.1, IC1.VBB1, IC1.VBB2, IC5.VI
- net X-DIR: no longer IC1.DIR
- net X-STEP: no longer IC1.STEP
Other:
- moved on the sheet: C46, C47, C48, C49, C50, C51, JP1, MS-X, R27, R28, R29, R30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
