File: melzi.sch (EAGLE design)
At the start: 124 parts, among them IC4 A4988, IC5 7805DT, IC6 ATMEGA644A, IC7 4050D, IC8 FT232RL-BASICSSOP, M1 RFP30N06LE, M2 RFP30N06LE, M3 RFP30N06LE, Q1 16MHZ, T4 TRIM, U1 A4982, U2 A4982, U3 A4982, X1 MICROSD, X2 MINI-USB-SHIELD-UX60-MB-5ST

Commit message: Pretty much finalised.  A couple of unrouted grounds need to be fixed.
Parts:
- removed C25, C40: .22uf, SparkFun:CAP0805
- removed C26: .33uf, SparkFun:CAP0805
- removed C39: .1uf, SparkFun:CAP0805
- removed IC4: A4988, allegro:A4983
- removed JS13: MS1, SparkFun:JUMPER-2SMD-NC
- removed JS14: MS2, SparkFun:JUMPER-2SMD-NC
- removed JS15: MS3, SparkFun:JUMPER-2SMD-NC
- removed S7, S8: 0.05, SparkFun:RESISTOR1206
- removed T4: TRIM, SparkFun:TRIMPOTSMD
- added C19: 0.22uF, ipc-7351-capacitor:CAPACITOR_0805
- added C20: 10uF, ipc-7351-capacitor:CAPACITOR_0805
- added C21: 0.1uF, ipc-7351-capacitor:CAPACITOR_0805
- added MS-X3: (no value), printrbot:SOLDERJUMPER_2WAYCONNECTED
- added R36: 100k, ipc-7351-resistor:RESISTOR_0805
- added R37: 4k7, ipc-7351-resistor:RESISTOR_0805
- added R38: 20k, ipc-7351-resistor:RESISTOR_0805
- added U4: A4982, printrbot:A4982
- C22: value .1uf -> 100uF; device SparkFun:CAP0805 -> rcl:CPOL-USD
- C23: value .1uf -> 0.1uF; device SparkFun:CAP0805 -> ipc-7351-capacitor:CAPACITOR_0805
- C24: value .1uf -> 4.7 uF; device SparkFun:CAP0805 -> rcl:CPOL-EUSMCC
- C4: value 100 uF -> 0.1uF; device rcl:CPOL-EUUD-6,3X7,7 -> ipc-7351-capacitor:CAPACITOR_0805
- IC6: value ATMEGA644A -> ATMEGA1284P
- R16, R32, R34: value 100k -> 4k7
- R22: value 100k -> 0.11; device SparkFun:RESISTOR -> ipc-7351-resistor:RESISTOR_0805
- R23: value 10k -> 0.11; device SparkFun:RESISTOR -> ipc-7351-resistor:RESISTOR_0805
- R24: device SparkFun:RESISTOR -> ipc-7351-resistor:RESISTOR_0805
- R9: value 20k -> 10k; device SparkFun:RESISTOR -> printrbot:RTRIM-ST-4EA
Connections:
- removed net EOUT1A: IC4.OUT1A, JP4.3
- removed net EOUT1B: IC4.OUT1B, JP4.4
- removed net EOUT2A: IC4.OUT2A, JP4.2
- removed net EOUT2B: IC4.OUT2B, JP4.1
- removed net N$24: IC4.MS2, JS14.1
- removed net XCP7: C22.1, IC4.CP1
- removed net XCP8: C22.2, IC4.CP2
- removed net XREF6: IC4.REF, T4.WIPER
- removed net XREF7: R9.2, T4.CW
- removed net XROSC3: IC4.ROSC, R23.1
- removed net XSENSE7: IC4.SENSE2, S7.2
- removed net XSENSE8: IC4.SENSE1, S8.2
- removed net XSLEEP3: IC4.RESET, IC4.SLEEP, R24.2
- removed net XVCP3: C39.2, IC4.VCP
- removed net XVREG3: C40.2, IC4.VREG
- new net N$60: R22.1, U4.SENSE1
- new net N$61: R23.1, U4.SENSE2
- new net N$62: R9.S, U4.REF
- new net N$63: R24.1, U4.ROSC
- new net N$64: C19.2, U4.VREG
- new net N$65: R37.2, U4.!RESET, U4.!SLEEP
- new net N$66: C21.2, U4.VCP
- new net N$67: MS-X3.1, U4.MS1
- new net N$68: MS-X3.3, U4.MS2
- new net N$70: JP4.3, U4.OUT1A
- new net N$71: JP4.4, U4.OUT1B
- new net N$72: JP4.2, U4.OUT2A
- new net N$73: JP4.1, U4.OUT2B
- new net N$74: R38.1, R9.A
- net !XYEENABLE: now also R36.2, U4.!ENABLE; no longer IC4.ENABLE, R22.2
- net E-DIR: now also U4.DIR; no longer IC4.DIR
- net E-STEP: now also U4.STEP; no longer IC4.STEP
- net GND: now also C19.1, C20.1, C22.-, C24.-, R22.2, R24.2, R9.E, U4.GND1, U4.GND2, U4.PAD; no longer C24.1, C25.2, C26.2, C4.-, C40.1, IC4.EXP, IC4.GND, IC4.GND@1, IC4.NC, IC4.NC@1, IC4.NC@2, S7.1, S8.1, T4.CCW
- net N$25: now also C4.2, U4.CP1; no longer IC4.MS3, JS15.1
- net N$27: now also C4.1, U4.CP2; no longer IC4.MS1, JS13.1
- net N$36: now also C24.+; no longer C26.1
- net VCC: now also C20.2, MS-X3.2, R36.1, R37.1, R38.2, U4.VDD; no longer C25.1, IC4.VDD, JS13.2, JS14.2, JS15.2, R22.1, R24.1, R9.1
- net VMOT: now also C21.1, C22.+, U4.VBB1, U4.VBB2; no longer C24.2, C39.1, C4.+, IC4.VBB1, IC4.VBB2
Other:
- note added: "Motor Control E"
- note added: "Motor Control Z"
- moved on the sheet: C23, JP4

Commit message: Melzi 2.0 finished (e&oe...)
Parts:
- JP4: value Y-MOT -> E-MOT
Changed lines of the file:
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@@
 <part name="JP2" library="SparkFun" deviceset="M04" device="SCREW" value="Y-MOT"/>
 <part name="JP3" library="SparkFun" deviceset="M04" device="SCREW" value="Z-MOT"/>
-<part name="JP4" library="SparkFun" deviceset="M04" device="SCREW" value="Y-MOT"/>
+<part name="JP4" library="SparkFun" deviceset="M04" device="SCREW" value="E-MOT"/>
 <part name="Q1" library="murata-filter" deviceset="CSTCR" device="" technology="6M00G53Z" value="16MHZ"/>
 <part name="X2" library="con-hirose" deviceset="MINI-USB-SHIELD-" device="UX60-MB-5ST"/>

Commit message: Thermistor resistors changed to 4K7.
Parts:
- R4, R5: value 10k -> 4k7
Changed lines of the file:
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@@
 <part name="R12" library="SparkFun" deviceset="RESISTOR" device="1206" value="10k"/>
 <part name="GND74" library="SparkFun" deviceset="GND" device=""/>
-<part name="R4" library="SparkFun" deviceset="RESISTOR" device="1206" value="10k"/>
+<part name="R4" library="SparkFun" deviceset="RESISTOR" device="1206" value="4k7"/>
 <part name="C8" library="rcl" deviceset="CPOL-EU" device="SMCC" value="4.7 uF"/>
 <part name="GND77" library="SparkFun" deviceset="GND" device=""/>
 <part name="P+21" library="supply1" deviceset="VCC" device=""/>
-<part name="R5" library="SparkFun" deviceset="RESISTOR" device="1206" value="10k"/>
+<part name="R5" library="SparkFun" deviceset="RESISTOR" device="1206" value="4k7"/>
 <part name="C9" library="rcl" deviceset="CPOL-EU" device="SMCC" value="4.7 uF"/>
 <part name="GND78" library="SparkFun" deviceset="GND" device=""/>

Commit message: Made motor current pots turn the right way.
Connections:
- net GND: now also R27.A, R6.A, R8.A, R9.A; no longer R27.E, R6.E, R8.E, R9.E
- net N$46: now also R6.E; no longer R6.A
- net N$59: now also R8.E; no longer R8.A
- net N$69: now also R27.E; no longer R27.A
- net N$74: now also R9.E; no longer R9.A
Other:
- moved on the sheet: R27, R6, R8, R9
Changed lines of the file:
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@@
 <instance part="JS2" gate="A" x="401.32" y="167.64" rot="R90"/>
 <instance part="JS3" gate="A" x="447.04" y="167.64" rot="R90"/>
-<instance part="R27" gate="G$1" x="228.6" y="218.44"/>
+<instance part="R27" gate="G$1" x="228.6" y="218.44" rot="MR180"/>
 <instance part="U2" gate="G$1" x="269.24" y="241.3"/>
 <instance part="C46" gate="G$1" x="269.24" y="271.78" rot="R180"/>
@@
 <instance part="P+19" gate="VCC" x="238.76" y="264.16"/>
 <instance part="U$1" gate="G$1" x="414.02" y="261.62"/>
-<instance part="R6" gate="G$1" x="342.9" y="218.44"/>
+<instance part="R6" gate="G$1" x="342.9" y="218.44" rot="MR180"/>
 <instance part="U1" gate="G$1" x="383.54" y="241.3"/>
 <instance part="C1" gate="G$1" x="383.54" y="271.78" rot="R180"/>
@@
 <instance part="P+1" gate="VCC" x="353.06" y="264.16"/>
 <instance part="U$2" gate="G$1" x="525.78" y="261.62"/>
-<instance part="R8" gate="G$1" x="454.66" y="218.44"/>
+<instance part="R8" gate="G$1" x="454.66" y="218.44" rot="MR180"/>
 <instance part="U3" gate="G$1" x="495.3" y="241.3"/>
 <instance part="C3" gate="G$1" x="495.3" y="271.78" rot="R180"/>
@@
 <instance part="P+2" gate="VCC" x="464.82" y="264.16"/>
 <instance part="U$3" gate="G$1" x="637.54" y="261.62"/>
-<instance part="R9" gate="G$1" x="566.42" y="218.44"/>
+<instance part="R9" gate="G$1" x="566.42" y="218.44" rot="MR180"/>
 <instance part="U4" gate="G$1" x="607.06" y="241.3"/>
 <instance part="C4" gate="G$1" x="607.06" y="271.78" rot="R180"/>
@@
 <wire x1="251.46" y1="220.98" x2="248.92" y2="220.98" width="0.1524" layer="91"/>
 <wire x1="251.46" y1="218.44" x2="248.92" y2="218.44" width="0.1524" layer="91"/>
-<wire x1="228.6" y1="213.36" x2="248.92" y2="213.36" width="0.1524" layer="91"/>
 <wire x1="248.92" y1="213.36" x2="248.92" y2="218.44" width="0.1524" layer="91"/>
 <junction x="248.92" y="220.98"/>
@@
 <pinref part="U2" gate="G$1" pin="PAD"/>
 <pinref part="GND65" gate="1" pin="GND"/>
-<pinref part="R27" gate="G$1" pin="E"/>
+<pinref part="R27" gate="G$1" pin="A"/>
+<wire x1="228.6" y1="213.36" x2="248.92" y2="213.36" width="0.1524" layer="91"/>
+<junction x="248.92" y="213.36"/>
 </segment>
 <segment>
@@
 <wire x1="365.76" y1="220.98" x2="363.22" y2="220.98" width="0.1524" layer="91"/>
 <wire x1="365.76" y1="218.44" x2="363.22" y2="218.44" width="0.1524" layer="91"/>
-<wire x1="342.9" y1="213.36" x2="363.22" y2="213.36" width="0.1524" layer="91"/>
 <wire x1="363.22" y1="213.36" x2="363.22" y2="218.44" width="0.1524" layer="91"/>
 <junction x="363.22" y="220.98"/>
@@
 <pinref part="U1" gate="G$1" pin="PAD"/>
 <pinref part="GND2" gate="1" pin="GND"/>
-<pinref part="R6" gate="G$1" pin="E"/>
+<pinref part="R6" gate="G$1" pin="A"/>
+<wire x1="342.9" y1="213.36" x2="363.22" y2="213.36" width="0.1524" layer="91"/>
+<junction x="363.22" y="213.36"/>
 </segment>
 <segment>
@@
 <wire x1="477.52" y1="220.98" x2="474.98" y2="220.98" width="0.1524" layer="91"/>
 <wire x1="477.52" y1="218.44" x2="474.98" y2="218.44" width="0.1524" layer="91"/>
-<wire x1="454.66" y1="213.36" x2="474.98" y2="213.36" width="0.1524" layer="91"/>
 <wire x1="474.98" y1="213.36" x2="474.98" y2="218.44" width="0.1524" layer="91"/>
 <junction x="474.98" y="220.98"/>
@@
 <pinref part="U3" gate="G$1" pin="PAD"/>
 <pinref part="GND8" gate="1" pin="GND"/>
-<pinref part="R8" gate="G$1" pin="E"/>
+<pinref part="R8" gate="G$1" pin="A"/>
+<wire x1="454.66" y1="213.36" x2="474.98" y2="213.36" width="0.1524" layer="91"/>
+<junction x="474.98" y="213.36"/>
 </segment>
 <segment>
@@
 <wire x1="589.28" y1="220.98" x2="586.74" y2="220.98" width="0.1524" layer="91"/>
 <wire x1="589.28" y1="218.44" x2="586.74" y2="218.44" width="0.1524" layer="91"/>
-<wire x1="566.42" y1="213.36" x2="586.74" y2="213.36" width="0.1524" layer="91"/>
 <wire x1="586.74" y1="213.36" x2="586.74" y2="218.44" width="0.1524" layer="91"/>
 <junction x="586.74" y="220.98"/>
@@
 <pinref part="U4" gate="G$1" pin="PAD"/>
 <pinref part="GND14" gate="1" pin="GND"/>
-<pinref part="R9" gate="G$1" pin="E"/>
+<pinref part="R9" gate="G$1" pin="A"/>
+<wire x1="566.42" y1="213.36" x2="586.74" y2="213.36" width="0.1524" layer="91"/>
+<junction x="586.74" y="213.36"/>
 </segment>
 <segment>
@@
 <net name="N$7" class="0">
 <segment>
-<wire x1="233.68" y1="218.44" x2="241.3" y2="218.44" width="0.1524" layer="91"/>
 <wire x1="241.3" y1="218.44" x2="241.3" y2="228.6" width="0.1524" layer="91"/>
 <wire x1="241.3" y1="228.6" x2="251.46" y2="228.6" width="0.1524" layer="91"/>
+<pinref part="U2" gate="G$1" pin="REF"/>
 <pinref part="R27" gate="G$1" pin="S"/>
-<pinref part="U2" gate="G$1" pin="REF"/>
+<wire x1="241.3" y1="218.44" x2="233.68" y2="218.44" width="0.1524" layer="91"/>
 </segment>
 </net>
@@
 <wire x1="287.02" y1="241.3" x2="294.64" y2="241.3" width="0.1524" layer="91"/>
 <junction x="294.64" y="241.3"/>
-</segment>
-</net>
-<net name="N$69" class="0">
-<segment>
-<pinref part="R39" gate="G$1" pin="1"/>
-<pinref part="R27" gate="G$1" pin="A"/>
 </segment>
 </net>
@@
 <net name="N$18" class="0">
 <segment>
-<wire x1="347.98" y1="218.44" x2="355.6" y2="218.44" width="0.1524" layer="91"/>
 <wire x1="355.6" y1="218.44" x2="355.6" y2="228.6" width="0.1524" layer="91"/>
 <wire x1="355.6" y1="228.6" x2="365.76" y2="228.6" width="0.1524" layer="91"/>
+<pinref part="U1" gate="G$1" pin="REF"/>
 <pinref part="R6" gate="G$1" pin="S"/>
-<pinref part="U1" gate="G$1" pin="REF"/>
+<wire x1="347.98" y1="218.44" x2="355.6" y2="218.44" width="0.1524" layer="91"/>
 </segment>
 </net>
@@
 </segment>
 </net>
-<net name="N$46" class="0">
-<segment>
-<pinref part="R17" gate="G$1" pin="1"/>
-<pinref part="R6" gate="G$1" pin="A"/>
-</segment>
-</net>
 <net name="N$20" class="0">
 <segment>
@@
 <net name="N$48" class="0">
 <segment>
-<wire x1="459.74" y1="218.44" x2="467.36" y2="218.44" width="0.1524" layer="91"/>
 <wire x1="467.36" y1="218.44" x2="467.36" y2="228.6" width="0.1524" layer="91"/>
 <wire x1="467.36" y1="228.6" x2="477.52" y2="228.6" width="0.1524" layer="91"/>
+<pinref part="U3" gate="G$1" pin="REF"/>
 <pinref part="R8" gate="G$1" pin="S"/>
-<pinref part="U3" gate="G$1" pin="REF"/>
+<wire x1="467.36" y1="218.44" x2="459.74" y2="218.44" width="0.1524" layer="91"/>
 </segment>
 </net>
@@
 </segment>
 </net>
-<net name="N$59" class="0">
-<segment>
-<pinref part="R35" gate="G$1" pin="1"/>
-<pinref part="R8" gate="G$1" pin="A"/>
-</segment>
-</net>
 <net name="N$24" class="0">
 <segment>
@@
 </segment>
 </net>
+<net name="N$75" class="0">
+<segment>
+<wire x1="662.94" y1="259.08" x2="662.94" y2="264.16" width="0.1524" layer="91"/>
+</segment>
+</net>
+<net name="N$69" class="0">
+<segment>
+<pinref part="R39" gate="G$1" pin="1"/>
+<pinref part="R27" gate="G$1" pin="E"/>
+<junction x="228.6" y="223.52"/>
+</segment>
+</net>
+<net name="N$46" class="0">
+<segment>
+<pinref part="R17" gate="G$1" pin="1"/>
+<pinref part="R6" gate="G$1" pin="E"/>
+<junction x="342.9" y="223.52"/>
+</segment>
+</net>
+<net name="N$59" class="0">
+<segment>
+<pinref part="R35" gate="G$1" pin="1"/>
+<pinref part="R8" gate="G$1" pin="E"/>
+<junction x="454.66" y="223.52"/>
+</segment>
+</net>
 <net name="N$74" class="0">
 <segment>
 <pinref part="R38" gate="G$1" pin="1"/>
-<pinref part="R9" gate="G$1" pin="A"/>
-</segment>
-</net>
-<net name="N$75" class="0">
-<segment>
-<wire x1="662.94" y1="259.08" x2="662.94" y2="264.16" width="0.1524" layer="91"/>
-</segment>
-</net>
+<pinref part="R9" gate="G$1" pin="E"/>
+<junction x="566.42" y="223.52"/>
+</segment>
+</net>

Commit message: Added 0.33uF upstream of 5V reg.  Specified 4.7uF cap in parallel as 30V.
Parts:
- added C25: .33uf, SparkFun:CAP0805
- C24: value 4.7 uF -> 4.7 uF 30V
Connections:
- net GND: now also C25.2
- net N$36: now also C25.1
Changed lines of the file:
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@@
 <part name="R38" library="ipc-7351-resistor" deviceset="RESISTOR_" device="0805" value="20k"/>
 <part name="P+3" library="supply1" deviceset="VCC" device=""/>
-<part name="C24" library="rcl" deviceset="CPOL-EU" device="SMCC" value="4.7 uF"/>
+<part name="C24" library="rcl" deviceset="CPOL-EU" device="SMCC" value="4.7 uF 30V"/>
+<part name="C25" library="SparkFun" deviceset="CAP" device="0805" value=".33uf"/>
 </parts>
 <sheets>
@@
 <instance part="P+3" gate="VCC" x="576.58" y="264.16"/>
 <instance part="C24" gate="G$1" x="281.94" y="160.02"/>
+<instance part="C25" gate="G$1" x="274.32" y="157.48"/>
 </instances>
 <busses>
@@
 <pinref part="GND75" gate="1" pin="GND"/>
 <pinref part="C24" gate="G$1" pin="-"/>
+<pinref part="C25" gate="G$1" pin="2"/>
+<wire x1="281.94" y1="154.94" x2="274.32" y2="154.94" width="0.1524" layer="91"/>
 </segment>
 <segment>
@@
 <pinref part="C24" gate="G$1" pin="+"/>
 <junction x="281.94" y="162.56"/>
-</segment>
-</net>
+<pinref part="C25" gate="G$1" pin="1"/>
+<wire x1="281.94" y1="162.56" x2="274.32" y2="162.56" width="0.1524" layer="91"/>
+</segment>
+</net>
