File: Kicad2/melzi.sch (EAGLE design)
At the start: 121 parts, among them IC5 7805DT, IC6 ATMEGA644A, IC7 4050D, IC8 FT232RL-BASICSSOP, M1 RFP30N06LE, M2 RFP30N06LE, M3 RFP30N06LE, Q1 16MHZ, U1 A4982, U2 A4982, U3 A4982, U4 A4982, X1 MICROSD, X2 MINI-USB-SHIELD-UX60-MB-5ST

Commit message: "Made in the UK" added to silkscreen.
Parts:
- removed C26: .33uf, SparkFun:CAP0805
- added C24: 4.7 uF 30V, rcl:CPOL-EUSMCC
- added C25: .33uf, SparkFun:CAP0805
- IC6: value ATMEGA644A -> ATMEGA1284P
- JP4: value Y-MOT -> E-MOT
- R4, R5: value 10k -> 4k7
Connections:
- net GND: now also C24.-, C25.2, R27.A, R6.A, R8.A, R9.A; no longer C26.2, R27.E, R6.E, R8.E, R9.E
- net N$36: now also C24.+, C25.1; no longer C26.1
- net N$46: now also R6.E; no longer R6.A
- net N$59: now also R8.E; no longer R8.A
- net N$69: now also R27.E; no longer R27.A
- net N$74: now also R9.E; no longer R9.A
Other:
- moved on the sheet: R27, R6, R8, R9
